Commit message: [E1] La columna dejaba de atravesar el eslabon 1
El eslabon 1 va centrado en el eje de theta1, de modo que su mitad inferior
quedaba dentro del volumen de la columna, que llegaba hasta el propio eje. Dos
solidos compartiendo espacio no es fabricable y falsea las propiedades masicas.

Ademas sus caras superiores quedaban coplanarias, y al seleccionar una en
Fusion se obtenia la otra: al intentar la union de theta1 se seleccionaba dos
veces el mismo componente y Fusion respondia que estaban ensamblados de forma
rigida.

La columna termina ahora en la cara inferior del eslabon, que es donde apoyaria
el rodamiento. El motor de theta1 acompana ese cambio y sigue alojado en su
interior.

File: src/station1_description/urdf/station1.urdf.xacro (robot description, xacro)
@@ -36,5 +36,5 @@
   =================================================================== -->
   <xacro:property name="m_placa"   value="${densidad_mdf * base_x * base_y * base_z}"/>
-  <xacro:property name="m_columna" value="${densidad_pla * pi * columna_radio * columna_radio * (altura_columna - base_z)}"/>
+  <xacro:property name="m_columna" value="${densidad_pla * pi * columna_radio * columna_radio * (altura_columna - brazo_espesor/2 - base_z)}"/>
   <xacro:property name="m_base"    value="${m_placa + m_columna + motor_masa}"/>
   <link name="${p}base_link">
@@ -44,7 +44,9 @@
       <material name="mdf"/>
     </visual>
-    <visual>
-      <origin xyz="0 0 ${base_z + (altura_columna - base_z)/2}"/>
-      <geometry><cylinder radius="${columna_radio}" length="${altura_columna - base_z}"/></geometry>
+    <!-- La columna termina en la cara inferior del eslabon 1, que es donde
+         apoya el rodamiento de theta1. -->
+    <visual>
+      <origin xyz="0 0 ${base_z + (altura_columna - brazo_espesor/2 - base_z)/2}"/>
+      <geometry><cylinder radius="${columna_radio}" length="${altura_columna - brazo_espesor/2 - base_z}"/></geometry>
       <material name="pla"/>
     </visual>
@@ -54,6 +56,6 @@
     </collision>
     <collision>
-      <origin xyz="0 0 ${base_z + (altura_columna - base_z)/2}"/>
-      <geometry><cylinder radius="${columna_radio}" length="${altura_columna - base_z}"/></geometry>
+      <origin xyz="0 0 ${base_z + (altura_columna - brazo_espesor/2 - base_z)/2}"/>
+      <geometry><cylinder radius="${columna_radio}" length="${altura_columna - brazo_espesor/2 - base_z}"/></geometry>
     </collision>
     <inertial>

Commit message: [E1] La tuerca deja de sobresalir por encima del husillo
Estaba dibujada a caballo sobre el extremo del husillo, sobresaliendo 7.5 mm.
El punto mas alto de la estacion pasaba a ser la tuerca, a 314.5 mm, y no el
husillo a 307, que es lo que estaba documentado.

Se queda dentro del limite de 320 mm, pero el margen bajaba de 13 a 5.5 mm, y
ahi todavia falta alojar el rodamiento superior del husillo. La tuerca cuelga
ahora del extremo sin sobresalir.

File: src/station1_description/urdf/station1.urdf.xacro (robot description, xacro)
@@ -223,6 +223,8 @@
   <xacro:property name="cz_link3"  value="${(tuerca_masa*0.0 + m_vastago*(-vastago_largo/2))/m_link3}"/>
   <link name="${p}link_3">
-    <visual>
-      <origin xyz="0 0 0"/>
+    <!-- La tuerca cuelga del extremo del husillo, sin sobresalir por encima:
+         el punto mas alto de la estacion debe ser el husillo, no ella. -->
+    <visual>
+      <origin xyz="0 0 ${-tuerca_lado/4}"/>
       <geometry><box size="${tuerca_lado} ${tuerca_lado} ${tuerca_lado/2}"/></geometry>
       <material name="metal"/>
