Commit message: [E1] Arquitectura de transmision por correa y actuadores en el modelo
El modelo no incluia los actuadores: solo tenia los eslabones estructurales,
de modo que el brazo estaba dimensionado como si los motores no pesaran ni
ocuparan sitio. Medidos sobre el CAD del fabricante, los Pololu 37D son de
37 mm de diametro y 82 mm de largo, con unos 200 g de masa cada uno.

Montados directamente sobre las articulaciones rompian dos cosas: la altura,
porque el motor de la prismatica apilado sobre el husillo daba 374 mm frente a
los 320 de maximo, y el equilibrio, porque dejaba 400 g en voladizo sobre unos
eslabones de acrilico de 85 g.

Se adopta la solucion estandar en SCARA:

  theta1  motor alojado dentro de la columna, accionamiento directo
  theta2  motor en la base, correa dentada por dentro del eslabon 1
  d3      motor en el codo, correa al husillo del extremo del eslabon 2

Dos de los tres motores quedan fijos a la base. El eje vertical pasa a ser un
husillo fijo al eslabon 2 con la tuerca desplazandose sobre el, de modo que la
altura maxima ya no depende de la posicion del efector.

La masa del modelo pasa de 543 g a 1947 g, que es la que corresponde. El
eslabon 2 lleva inercia compuesta por el teorema de Steiner, con su producto
de inercia, al cargar el motor descentrado.

Verificado: altura 307 mm, alcance de los seis puntos de tarea, arbol TF
correcto y modelo spawneado en el mundo.

File: src/station1_description/urdf/parametros.xacro (robot description, xacro)
@@ -7,4 +7,9 @@
   geometria y la densidad del material asignado.
   Unidades del Sistema Internacional: metros, kilogramos, radianes, segundos.
+  Revision del 13 de agosto de 2026: arquitectura de transmision por correa.
+  Los motores Pololu 37D miden 37 mm de diametro y pesan del orden de 200 g
+  cada uno. Montados directamente sobre las articulaciones rompian la
+  restriccion de altura y dejaban dos tercios de la masa en voladizo, de modo
+  que los dos motores rotacionales pasan a la base y accionan por correa.
 -->
 <robot xmlns:xacro="http://www.ros.org/wiki/xacro">
@@ -21,50 +26,82 @@
   <xacro:property name="l1" value="0.180"/>   <!-- eslabon 1, brazo    -->
   <xacro:property name="l2" value="0.140"/>   <!-- eslabon 2, antebrazo-->
-  <!-- Altura del plano del brazo y carrera vertical.
-       El eje de la prismatica sobresale por encima del brazo cuando el efector
-       baja, de modo que la altura maxima de la estacion es la suma de ambas:
-       0.180 + 0.120 = 0.300 m, que es exactamente el valor nominal exigido.
-       El efector recorre entonces z de 0.145 a 0.025, y los puntos de tarea
-       estan a 0.050 y 0.060. -->
-  <xacro:property name="altura_columna" value="0.180"/>
+  <!-- Altura del plano del brazo. La columna aloja en su interior el
+       motor de theta1, de modo que debe ser mas alta que el propio motor. -->
+  <xacro:property name="altura_columna" value="0.170"/>
+  <!-- ================== Eje vertical d3 ===========================
+       Husillo fijo al eslabon 2, con la tuerca desplazandose sobre el. El
+       efector cuelga de la tuerca mediante un vastago guiado. La altura
+       maxima de la estacion la fija el extremo del husillo, que no se mueve:
+       altura_columna - brazo_espesor + husillo_largo.
+  -->
+  <xacro:property name="husillo_largo"  value="0.145"/>  <!-- carrera mas tuerca y rodamiento -->
+  <xacro:property name="husillo_radio"  value="0.004"/>  <!-- T8, 8 mm de diametro -->
   <xacro:property name="carrera_d3"     value="0.120"/>
+  <xacro:property name="vastago_largo"  value="0.150"/>
+  <xacro:property name="vastago_radio"  value="0.008"/>
+  <xacro:property name="tuerca_lado"    value="0.030"/>
   <!-- ================== Limites de articulacion ==================== -->
   <xacro:property name="lim_theta1" value="2.618"/>   <!-- +/- 150 grados -->
   <xacro:property name="lim_theta2" value="2.356"/>   <!-- +/- 135 grados -->
   <xacro:property name="lim_gripper" value="0.500"/>
-  <!-- Velocidad maxima de las articulaciones rotacionales.            -->
-  <!-- Motor Pololu de 200 RPM: 200 * 2*pi / 60 = 20.944 rad/s en el   -->
-  <!-- eje de salida, sin reduccion adicional.                          -->
-  <xacro:property name="vel_rot" value="20.944"/>
-  <!-- Velocidad de la articulacion prismatica. Husillo T8 de 8 mm de  -->
-  <!-- avance por vuelta: 200/60 rev/s * 0.008 m = 0.0267 m/s.          -->
+  <!-- Velocidad de las articulaciones rotacionales.
+       Motor Pololu de 200 RPM: 200 * 2*pi / 60 = 20.944 rad/s en el eje de
+       salida. La transmision por correa es de relacion 1:1, de modo que la
+       articulacion gira a la misma velocidad. -->
+  <xacro:property name="relacion_correa" value="1.0"/>
+  <xacro:property name="vel_rot" value="${20.944 / relacion_correa}"/>
+  <!-- Velocidad de la articulacion prismatica. Husillo T8 de 8 mm de
+       avance por vuelta: 200/60 rev/s * 0.008 m = 0.0267 m/s. -->
   <xacro:property name="avance_husillo" value="0.008"/>
   <xacro:property name="vel_pris" value="0.0267"/>
-  <!-- PROVISIONAL. El par disponible en el eje de salida debe tomarse  -->
-  <!-- de la hoja de datos del motor antes de la Entrega 2, junto con   -->
-  <!-- el calculo del par requerido por cada articulacion.              -->
+  <!-- PROVISIONAL. El par disponible debe tomarse de la hoja de datos del
+       motor y contrastarse con el par requerido por cada articulacion. -->
   <xacro:property name="esfuerzo_rot"  value="0.50"/>   <!-- N.m  -->
   <xacro:property name="esfuerzo_pris" value="20.0"/>   <!-- N    -->
+  <!-- ================== Actuadores ================================
+       Envolvente medida sobre el modelo CAD del fabricante. La masa procede
+       de la hoja de datos y debe confirmarse con la referencia exacta que
+       entregue el laboratorio: la version con reductora es mas larga.
+  -->
+  <xacro:property name="motor_diametro" value="0.037"/>
+  <xacro:property name="motor_largo"    value="0.082"/>
+  <xacro:property name="motor_masa"     value="0.200"/>
+  <!-- Micro servo Tower Pro 9 g -->
+  <xacro:property name="servo_x"    value="0.023"/>
+  <xacro:property name="servo_y"    value="0.012"/>
+  <xacro:property name="servo_z"    value="0.029"/>
+  <xacro:property name="masa_servo" value="0.009"/>
+  <!-- Mordaza impresa que sujeta la pieza -->
+  <xacro:property name="gripper_x" value="0.040"/>
+  <xacro:property name="gripper_y" value="0.030"/>
+  <xacro:property name="gripper_z" value="0.035"/>
   <!-- ================== Materiales ================================ -->
   <!-- Densidades reales, usadas para derivar masas e inercias.        -->
-  <xacro:property name="densidad_mdf"     value="700.0"/>    <!-- kg/m3 -->
+  <xacro:property name="densidad_mdf"      value="700.0"/>   <!-- kg/m3 -->
   <xacro:property name="densidad_acrilico" value="1180.0"/>  <!-- kg/m3 -->
-  <xacro:property name="densidad_pla"     value="1240.0"/>   <!-- kg/m3 -->
+  <xacro:property name="densidad_pla"      value="1240.0"/>  <!-- kg/m3 -->
+  <xacro:property name="densidad_acero"    value="7850.0"/>  <!-- kg/m3 -->
+  <xacro:property name="densidad_aluminio" value="2700.0"/>  <!-- kg/m3 -->
+  <!-- Componentes comerciales de la transmision. Masas aproximadas, a
+       confirmar al comprarlos. -->
+  <xacro:property name="polea_masa"  value="0.020"/>  <!-- polea dentada de aluminio -->
+  <xacro:property name="tuerca_masa" value="0.030"/>  <!-- tuerca de laton del husillo -->
   <!-- ================== Geometria de las piezas ==================== -->
-  <!-- Base: placa de MDF de 12 mm -->
-  <xacro:property name="base_x" value="0.200"/>
-  <xacro:property name="base_y" value="0.200"/>
+  <!-- Base: placa de MDF de 12 mm. Aloja los dos motores rotacionales. -->
+  <xacro:property name="base_x" value="0.220"/>
+  <xacro:property name="base_y" value="0.220"/>
   <xacro:property name="base_z" value="0.012"/>
-  <!-- Columna: tubo de PLA impreso -->
+  <!-- Columna: tubo que aloja el motor de theta1 -->
   <xacro:property name="columna_radio" value="0.030"/>
+  <!-- Posicion del motor de theta2 en la base, junto a la columna -->
+  <xacro:property name="motor2_offset" value="0.060"/>
   <!-- Eslabones del brazo: acrilico cortado por laser, 8 mm -->
   <xacro:property name="brazo_ancho"   value="0.050"/>
   <xacro:property name="brazo_espesor" value="0.008"/>
-  <!-- Eje vertical de la prismatica: varilla de PLA -->
-  <xacro:property name="eje_radio" value="0.010"/>
-  <!-- Efector final: micro servo Tower Pro 9 g mas mordaza impresa -->
-  <xacro:property name="gripper_x" value="0.040"/>
-  <xacro:property name="gripper_y" value="0.030"/>
-  <xacro:property name="gripper_z" value="0.035"/>
-  <xacro:property name="masa_servo" value="0.009"/>
+  <!-- Altura del efector alcanzable, derivada de la cadena vertical.
+       z_tool = altura_columna - brazo_espesor + husillo_largo
+                - vastago_largo - gripper_z - d3                         -->
+  <xacro:property name="z_tool_max"
+    value="${altura_columna - brazo_espesor + husillo_largo - vastago_largo - gripper_z}"/>
+  <xacro:property name="z_tool_min" value="${z_tool_max - carrera_d3}"/>
 </robot>

File: src/station1_description/urdf/station1.urdf.xacro (robot description, xacro)
@@ -5,7 +5,15 @@
   como desplazamiento vertical.
   Responsable: Santiago Fernando Machado Sanchez
-  La geometria vive en parametros.xacro y las propiedades inerciales se derivan
-  de ella mediante las macros de inercias.xacro. Al sustituir las dimensiones
-  por las del CAD definitivo, masas e inercias se recalculan solas.
+  Arquitectura de transmision por correa. Los motores Pololu 37D pesan del
+  orden de 200 g y miden 37 mm de diametro, de modo que montarlos sobre las
+  articulaciones rompia la restriccion de altura y dejaba la mayor parte de la
+  masa en voladizo:
+    theta1  motor alojado dentro de la columna, accionamiento directo
+    theta2  motor en la base, correa dentada por dentro del eslabon 1
+    d3      motor en el codo, correa al husillo del extremo del eslabon 2
+  Dos de los tres motores quedan fijos a la base y no cargan el brazo.
+  El eje vertical es un husillo fijo al eslabon 2, con la tuerca desplazandose
+  sobre el; el efector cuelga de la tuerca mediante un vastago guiado. La
+  altura maxima de la estacion la fija el extremo del husillo, que no se mueve.
   Todos los frames llevan el prefijo de la estacion, segun ADR-005.
 -->
@@ -20,7 +28,14 @@
   <material name="pla">       <color rgba="0.90 0.90 0.90 1.0"/></material>
   <material name="metal">     <color rgba="0.55 0.55 0.58 1.0"/></material>
-  <!-- ==================== base_link ====================
-       Placa de MDF de 12 mm y columna de PLA. Es un eslabon fijo, de modo que
-       su inercia no interviene en la dinamica; se declara por completitud. -->
+  <material name="motor">     <color rgba="0.20 0.20 0.22 1.0"/></material>
+  <!-- ==================================================================
+       base_link: placa de MDF, columna y los dos motores rotacionales.
+       Es un eslabon fijo al mundo, de modo que su inercia no interviene en
+       la dinamica; se declara con la masa real para que el balance total de
+       la estacion sea correcto.
+  =================================================================== -->
+  <xacro:property name="m_placa"   value="${densidad_mdf * base_x * base_y * base_z}"/>
+  <xacro:property name="m_columna" value="${densidad_pla * pi * columna_radio * columna_radio * (altura_columna - base_z)}"/>
+  <xacro:property name="m_base"    value="${m_placa + m_columna + 2 * motor_masa}"/>
   <link name="${p}base_link">
     <visual>
@@ -34,4 +49,11 @@
       <material name="pla"/>
     </visual>
+    <!-- Motor de theta2, en la base junto a la columna. Acciona el codo por
+         correa; su masa nunca viaja con el brazo. -->
+    <visual>
+      <origin xyz="${motor2_offset} 0 ${base_z + motor_largo/2}"/>
+      <geometry><cylinder radius="${motor_diametro/2}" length="${motor_largo}"/></geometry>
+      <material name="motor"/>
+    </visual>
     <collision>
       <origin xyz="0 0 ${base_z/2}"/>
@@ -42,7 +64,16 @@
       <geometry><cylinder radius="${columna_radio}" length="${altura_columna - base_z}"/></geometry>
     </collision>
-    <xacro:inercia_caja x="${base_x}" y="${base_y}" z="${base_z}" densidad="${densidad_mdf}">
-      <origin xyz="0 0 ${base_z/2}"/>
-    </xacro:inercia_caja>
+    <collision>
+      <origin xyz="${motor2_offset} 0 ${base_z + motor_largo/2}"/>
+      <geometry><cylinder radius="${motor_diametro/2}" length="${motor_largo}"/></geometry>
+    </collision>
+    <inertial>
+      <origin xyz="0 0 ${altura_columna/3}"/>
+      <mass value="${m_base}"/>
+      <inertia
+        ixx="${m_base * (base_y*base_y + altura_columna*altura_columna) / 12.0}" ixy="0.0" ixz="0.0"
+        iyy="${m_base * (base_x*base_x + altura_columna*altura_columna) / 12.0}" iyz="0.0"
+        izz="${m_base * (base_x*base_x + base_y*base_y) / 12.0}"/>
+    </inertial>
   </link>
   <!-- ==================== theta1: rotacion de la base ==================== -->
@@ -56,4 +87,7 @@
     <dynamics damping="0.05" friction="0.01"/>
   </joint>
+  <!-- link_1: pletina de acrilico mas las dos poleas de la correa de theta2 -->
+  <xacro:property name="m_barra1" value="${densidad_acrilico * l1 * brazo_ancho * brazo_espesor}"/>
+  <xacro:property name="m_link1"  value="${m_barra1 + 2 * polea_masa}"/>
   <link name="${p}link_1">
     <visual>
@@ -66,10 +100,16 @@
       <geometry><box size="${l1} ${brazo_ancho} ${brazo_espesor}"/></geometry>
     </collision>
-    <xacro:inercia_caja x="${l1}" y="${brazo_ancho}" z="${brazo_espesor}"
-                        densidad="${densidad_acrilico}">
+    <!-- Las poleas van en los dos extremos, de modo que el centro de masa
+         del conjunto sigue estando a media longitud. -->
+    <inertial>
       <origin xyz="${l1/2} 0 0"/>
-    </xacro:inercia_caja>
-  </link>
-  <!-- ==================== theta2: hombro ==================== -->
+      <mass value="${m_link1}"/>
+      <inertia
+        ixx="${m_barra1*(brazo_ancho*brazo_ancho + brazo_espesor*brazo_espesor)/12.0}" ixy="0.0" ixz="0.0"
+        iyy="${m_barra1*(l1*l1 + brazo_espesor*brazo_espesor)/12.0 + 2*polea_masa*(l1/2)*(l1/2)}" iyz="0.0"
+        izz="${m_barra1*(l1*l1 + brazo_ancho*brazo_ancho)/12.0 + 2*polea_masa*(l1/2)*(l1/2)}"/>
+    </inertial>
+  </link>
+  <!-- ==================== theta2: codo ==================== -->
   <joint name="${p}joint_2" type="revolute">
     <parent link="${p}link_1"/>
@@ -81,4 +121,28 @@
     <dynamics damping="0.05" friction="0.01"/>
   </joint>
+  <!-- link_2: pletina, motor de d3 sobre el codo y husillo en el extremo.
+       Es el unico eslabon que carga un motor, y va en el codo y no en el
+       extremo para reducir su brazo respecto del eje de theta1. -->
+  <xacro:property name="m_barra2"   value="${densidad_acrilico * l2 * brazo_ancho * brazo_espesor}"/>
+  <xacro:property name="m_husillo"  value="${densidad_acero * pi * husillo_radio * husillo_radio * husillo_largo}"/>
+  <xacro:property name="m_link2"    value="${m_barra2 + motor_masa + m_husillo}"/>
+  <!-- Posiciones de cada cuerpo dentro del eslabon -->
+  <xacro:property name="cx_barra2"  value="${l2/2}"/>
+  <xacro:property name="cx_motor2"  value="${motor_largo/2 + 0.010}"/>
+  <xacro:property name="cz_motor2"  value="${brazo_espesor/2 + motor_diametro/2}"/>
+  <xacro:property name="cx_husillo" value="${l2}"/>
+  <xacro:property name="cz_husillo" value="${husillo_largo/2}"/>
+  <!-- Centro de masa del conjunto -->
+  <xacro:property name="cx_link2"
+    value="${(m_barra2*cx_barra2 + motor_masa*cx_motor2 + m_husillo*cx_husillo)/m_link2}"/>
+  <xacro:property name="cz_link2"
+    value="${(motor_masa*cz_motor2 + m_husillo*cz_husillo)/m_link2}"/>
+  <!-- Desplazamientos respecto del centro de masa, para el teorema de Steiner -->
+  <xacro:property name="dx_b" value="${cx_barra2 - cx_link2}"/>
+  <xacro:property name="dz_b" value="${-cz_link2}"/>
+  <xacro:property name="dx_m" value="${cx_motor2 - cx_link2}"/>
+  <xacro:property name="dz_m" value="${cz_motor2 - cz_link2}"/>
+  <xacro:property name="dx_h" value="${cx_husillo - cx_link2}"/>
+  <xacro:property name="dz_h" value="${cz_husillo - cz_link2}"/>
   <link name="${p}link_2">
     <visual>
@@ -87,21 +151,48 @@
       <material name="acrilico"/>
     </visual>
+    <visual>
+      <origin xyz="${cx_motor2} 0 ${cz_motor2}" rpy="0 ${pi/2} 0"/>
+      <geometry><cylinder radius="${motor_diametro/2}" length="${motor_largo}"/></geometry>
+      <material name="motor"/>
+    </visual>
+    <visual>
+      <origin xyz="${l2} 0 ${husillo_largo/2}"/>
+      <geometry><cylinder radius="${husillo_radio}" length="${husillo_largo}"/></geometry>
+      <material name="metal"/>
+    </visual>
     <collision>
       <origin xyz="${l2/2} 0 0"/>
       <geometry><box size="${l2} ${brazo_ancho} ${brazo_espesor}"/></geometry>
     </collision>
-    <xacro:inercia_caja x="${l2}" y="${brazo_ancho}" z="${brazo_espesor}"
-                        densidad="${densidad_acrilico}">
-      <origin xyz="${l2/2} 0 0"/>
-    </xacro:inercia_caja>
+    <collision>
+      <origin xyz="${cx_motor2} 0 ${cz_motor2}" rpy="0 ${pi/2} 0"/>
+      <geometry><cylinder radius="${motor_diametro/2}" length="${motor_largo}"/></geometry>
+    </collision>
+    <inertial>
+      <origin xyz="${cx_link2} 0 ${cz_link2}"/>
+      <mass value="${m_link2}"/>
+      <inertia
+        ixx="${ m_barra2*(brazo_ancho*brazo_ancho + brazo_espesor*brazo_espesor)/12.0 + m_barra2*dz_b*dz_b
+              + motor_masa*(motor_diametro/2)*(motor_diametro/2)/2.0 + motor_masa*dz_m*dz_m
+              + m_husillo*(3*husillo_radio*husillo_radio + husillo_largo*husillo_largo)/12.0 + m_husillo*dz_h*dz_h }"
+        ixy="0.0"
+        ixz="${ -(m_barra2*dx_b*dz_b + motor_masa*dx_m*dz_m + m_husillo*dx_h*dz_h) }"
+        iyy="${ m_barra2*(l2*l2 + brazo_espesor*brazo_espesor)/12.0 + m_barra2*(dx_b*dx_b + dz_b*dz_b)
+              + motor_masa*(3*(motor_diametro/2)*(motor_diametro/2) + motor_largo*motor_largo)/12.0 + motor_masa*(dx_m*dx_m + dz_m*dz_m)
+              + m_husillo*(3*husillo_radio*husillo_radio + husillo_largo*husillo_largo)/12.0 + m_husillo*(dx_h*dx_h + dz_h*dz_h) }"
+        iyz="0.0"
+        izz="${ m_barra2*(l2*l2 + brazo_ancho*brazo_ancho)/12.0 + m_barra2*dx_b*dx_b
+              + motor_masa*(3*(motor_diametro/2)*(motor_diametro/2) + motor_largo*motor_largo)/12.0 + motor_masa*dx_m*dx_m
+              + m_husillo*(husillo_radio*husillo_radio)/2.0 + m_husillo*dx_h*dx_h }"/>
+    </inertial>
   </link>
   <!-- ==================== d3: desplazamiento vertical ====================
-       Accionada por husillo. El eje asciende por encima del brazo cuando el
-       efector desciende, de ahi que la altura maxima de la estacion sea la
-       suma de la columna y la carrera. -->
+       La tuerca recorre el husillo. El origen de la articulacion esta en el
+       extremo superior del husillo y el desplazamiento es descendente, de modo
+       que d3 = 0 corresponde al efector arriba. -->
   <joint name="${p}joint_3" type="prismatic">
     <parent link="${p}link_2"/>
     <child  link="${p}link_3"/>
-    <origin xyz="${l2} 0 0"/>
+    <origin xyz="${l2} 0 ${husillo_largo}"/>
     <axis xyz="0 0 -1"/>
     <limit lower="0.0" upper="${carrera_d3}"
@@ -109,30 +200,55 @@
     <dynamics damping="2.0" friction="0.5"/>
   </joint>
+  <!-- link_3: tuerca del husillo y vastago que sostiene el efector -->
+  <xacro:property name="m_vastago" value="${densidad_aluminio * pi * vastago_radio * vastago_radio * vastago_largo}"/>
+  <xacro:property name="m_link3"   value="${tuerca_masa + m_vastago}"/>
+  <xacro:property name="cz_link3"  value="${(tuerca_masa*0.0 + m_vastago*(-vastago_largo/2))/m_link3}"/>
   <link name="${p}link_3">
     <visual>
-      <origin xyz="0 0 ${carrera_d3/2}"/>
-      <geometry><cylinder radius="${eje_radio}" length="${carrera_d3}"/></geometry>
+      <origin xyz="0 0 0"/>
+      <geometry><box size="${tuerca_lado} ${tuerca_lado} ${tuerca_lado/2}"/></geometry>
       <material name="metal"/>
     </visual>
-    <collision>
-      <origin xyz="0 0 ${carrera_d3/2}"/>
-      <geometry><cylinder radius="${eje_radio}" length="${carrera_d3}"/></geometry>
-    </collision>
-    <xacro:inercia_cilindro radio="${eje_radio}" longitud="${carrera_d3}"
-                            densidad="${densidad_pla}">
-      <origin xyz="0 0 ${carrera_d3/2}"/>
-    </xacro:inercia_cilindro>
+    <visual>
+      <origin xyz="0 0 ${-vastago_largo/2}"/>
+      <geometry><cylinder radius="${vastago_radio}" length="${vastago_largo}"/></geometry>
+      <material name="metal"/>
+    </visual>
+    <collision>
+      <origin xyz="0 0 ${-vastago_largo/2}"/>
+      <geometry><cylinder radius="${vastago_radio}" length="${vastago_largo}"/></geometry>
+    </collision>
+    <inertial>
+      <origin xyz="0 0 ${cz_link3}"/>
+      <mass value="${m_link3}"/>
+      <inertia
+        ixx="${ tuerca_masa*(tuerca_lado*tuerca_lado + (tuerca_lado/2)*(tuerca_lado/2))/12.0 + tuerca_masa*cz_link3*cz_link3
+              + m_vastago*(3*vastago_radio*vastago_radio + vastago_largo*vastago_largo)/12.0
+              + m_vastago*(vastago_largo/2 + cz_link3)*(vastago_largo/2 + cz_link3) }"
+        ixy="0.0" ixz="0.0"
+        iyy="${ tuerca_masa*(tuerca_lado*tuerca_lado + (tuerca_lado/2)*(tuerca_lado/2))/12.0 + tuerca_masa*cz_link3*cz_link3
+              + m_vastago*(3*vastago_radio*vastago_radio + vastago_largo*vastago_largo)/12.0
+              + m_vastago*(vastago_largo/2 + cz_link3)*(vastago_largo/2 + cz_link3) }" iyz="0.0"
+        izz="${ tuerca_masa*(2*tuerca_lado*tuerca_lado)/12.0 + m_vastago*vastago_radio*vastago_radio/2.0 }"/>
+    </inertial>
   </link>
   <!-- ==================== Efector final ====================
        Micro servo Tower Pro 9 g con mordaza impresa. No cuenta como grado de
        libertad: los tres GDL son los tres motores DC. -->
+  <xacro:property name="m_mordaza" value="${densidad_pla * gripper_x * gripper_y * gripper_z * 0.35}"/>
+  <xacro:property name="m_gripper" value="${masa_servo + m_mordaza}"/>
   <joint name="${p}gripper_joint" type="revolute">
     <parent link="${p}link_3"/>
     <child  link="${p}gripper_link"/>
-    <origin xyz="0 0 0"/>
+    <origin xyz="0 0 ${-vastago_largo}"/>
     <axis xyz="1 0 0"/>
     <limit lower="0.0" upper="${lim_gripper}" velocity="3.0" effort="0.15"/>
   </joint>
   <link name="${p}gripper_link">
+    <visual>
+      <origin xyz="0 0 ${-servo_z/2}"/>
+      <geometry><box size="${servo_x} ${servo_y} ${servo_z}"/></geometry>
+      <material name="motor"/>
+    </visual>
     <visual>
       <origin xyz="0 0 ${-gripper_z/2}"/>
@@ -144,5 +260,5 @@
       <geometry><box size="${gripper_x} ${gripper_y} ${gripper_z}"/></geometry>
     </collision>
-    <xacro:inercia_componente masa="${masa_servo}"
+    <xacro:inercia_componente masa="${m_gripper}"
                               x="${gripper_x}" y="${gripper_y}" z="${gripper_z}">
       <origin xyz="0 0 ${-gripper_z/2}"/>
