Commit message: [E1] Ajusta el motor a la version con reductora
Medido sobre Gearmotor_37D_100.stp, que es el motor real: 94.6 mm de largo
total frente a los 81.6 del modelo anterior, que era la version sin reductora
y por tanto no alcanzaba las 200 RPM del enunciado.

Del mismo archivo salen las cotas de la interfaz mecanica, que condicionan el
diseno de las poleas y de los soportes: eje de salida de 6 mm, brida de
centraje de 16 mm y fijacion con tornilleria M3.

Holguras verificadas con el largo nuevo: el motor de theta1 deja 63 mm libres
dentro de la columna, el de theta2 queda 55 mm por debajo del plano del brazo
y el de d3 deja 35 mm hasta el husillo. La altura sigue en 307 mm.

File: src/station1_description/urdf/parametros.xacro (robot description, xacro)
@@ -60,11 +60,18 @@
   <xacro:property name="esfuerzo_pris" value="20.0"/>   <!-- N    -->
   <!-- ================== Actuadores ================================
-       Envolvente medida sobre el modelo CAD del fabricante. La masa procede
-       de la hoja de datos y debe confirmarse con la referencia exacta que
-       entregue el laboratorio: la version con reductora es mas larga.
+       Envolvente medida sobre Gearmotor_37D_100.stp, que es la version con
+       reductora: 94.6 mm de largo total y 36.8 mm de diametro de cuerpo. La
+       masa procede de la hoja de datos de Pololu y queda por confirmar contra
+       la referencia exacta que entregue el laboratorio.
   -->
   <xacro:property name="motor_diametro" value="0.037"/>
-  <xacro:property name="motor_largo"    value="0.082"/>
+  <xacro:property name="motor_largo"    value="0.095"/>
   <xacro:property name="motor_masa"     value="0.200"/>
+  <!-- Interfaz mecanica del motor, medida sobre Gearmotor_37D_100.stp.
+       Condiciona el diseno de las poleas, del acoplamiento al husillo y de
+       los soportes. -->
+  <xacro:property name="motor_eje_diametro"   value="0.006"/>
+  <xacro:property name="motor_brida_diametro" value="0.016"/>
+  <xacro:property name="motor_tornillo"       value="0.003"/>   <!-- M3 -->
   <!-- Micro servo Tower Pro 9 g -->
   <xacro:property name="servo_x"    value="0.023"/>

Commit message: [E1] Limites de esfuerzo derivados de la hoja de datos del motor
De la hoja de datos del Pololu 37D rev 1.2, la version de 200 RPM a 12 V es la
50:1, items #4743 sin encoder y #4753 con encoder. Longitud total 92.1 mm y
masa de 190 a 210 g; se toma el extremo superior.

El modelo CAD descargado corresponde a la version 100:1, cuya reductora es
2.5 mm mas larga: 94.6 frente a 92.1 mm.

El limite de par del modelo no lo fija el motor sino el driver. El 37D admite
100 kg.mm en continuo, 0.981 N.m, pero a ese par consume 2.72 A y el TB6612FNG
entrega 1.2 A continuos por canal. A esa corriente el motor da 39.6 kg.mm, de
modo que el limite util es 0.389 N.m, el 40 por ciento de lo que podria dar.

El esfuerzo de la prismatica se deriva del par por la relacion del husillo T8
en lugar de fijarse a mano: 61 N con rendimiento 0.2, frente a 1.4 N de carga
real.

Las articulaciones rotacionales tienen eje vertical y no levantan gravedad, de
modo que el par solo se emplea en acelerar. Esa es una de las razones de haber
elegido la configuracion RRP.

File: src/station1_description/urdf/parametros.xacro (robot description, xacro)
@@ -49,23 +49,36 @@
        salida. La transmision por correa es de relacion 1:1, de modo que la
        articulacion gira a la misma velocidad. -->
+  <xacro:property name="avance_husillo" value="0.008"/>
   <xacro:property name="relacion_correa" value="1.0"/>
   <xacro:property name="vel_rot" value="${20.944 / relacion_correa}"/>
   <!-- Velocidad de la articulacion prismatica. Husillo T8 de 8 mm de
        avance por vuelta: 200/60 rev/s * 0.008 m = 0.0267 m/s. -->
-  <xacro:property name="avance_husillo" value="0.008"/>
   <xacro:property name="vel_pris" value="0.0267"/>
-  <!-- PROVISIONAL. El par disponible debe tomarse de la hoja de datos del
-       motor y contrastarse con el par requerido por cada articulacion. -->
-  <xacro:property name="esfuerzo_rot"  value="0.50"/>   <!-- N.m  -->
-  <xacro:property name="esfuerzo_pris" value="20.0"/>   <!-- N    -->
+  <!-- Limites de esfuerzo, de la hoja de datos del 37D rev 1.2.
+       El motor admite 100 kg.mm en continuo, es decir 0.981 N.m, pero a ese
+       par consume 2.72 A y el driver TB6612FNG solo entrega 1.2 A continuos
+       por canal. Manda el driver: a 1.2 A el motor entrega 39.6 kg.mm.
+       El limite del modelo es por tanto el del sistema, no el del motor. -->
+  <xacro:property name="par_motor_continuo" value="0.981"/>  <!-- 100 kg.mm -->
+  <xacro:property name="par_motor_bloqueo"  value="2.059"/>  <!-- 210 kg.mm -->
+  <xacro:property name="esfuerzo_rot"       value="0.389"/>  <!-- limitado por el driver -->
+  <!-- Husillo T8: F = 2*pi*rendimiento*par/avance. Rendimiento 0.2, extremo
+       conservador de un husillo trapezoidal sin recirculacion de bolas. -->
+  <xacro:property name="rendimiento_husillo" value="0.2"/>
+  <xacro:property name="esfuerzo_pris"
+    value="${2 * pi * rendimiento_husillo * esfuerzo_rot / avance_husillo}"/>
   <!-- ================== Actuadores ================================
-       Envolvente medida sobre Gearmotor_37D_100.stp, que es la version con
-       reductora: 94.6 mm de largo total y 36.8 mm de diametro de cuerpo. La
-       masa procede de la hoja de datos de Pololu y queda por confirmar contra
-       la referencia exacta que entregue el laboratorio.
+       Pololu 37D 50:1 con encoder, item #4753, que a 12 V gira a 200 RPM sin
+       carga. Datos de la hoja de datos rev 1.2:
+         cuerpo de 36.8 mm de diametro y 92.1 mm de largo total
+         masa de 190 a 210 g; se toma el extremo superior
+         eje de salida de 6 mm y seis roscas M3 en circulo de 31 mm,
+         roscadas a 3 mm de profundidad como maximo
+       El modelo CAD descargado, Gearmotor_37D_100.stp, corresponde a la
+       version 100:1 y mide 94.6 mm: su reductora es 2.5 mm mas larga.
   -->
   <xacro:property name="motor_diametro" value="0.037"/>
-  <xacro:property name="motor_largo"    value="0.095"/>
-  <xacro:property name="motor_masa"     value="0.200"/>
+  <xacro:property name="motor_largo"    value="0.0921"/>
+  <xacro:property name="motor_masa"     value="0.210"/>
   <!-- Interfaz mecanica del motor, medida sobre Gearmotor_37D_100.stp.
        Condiciona el diseno de las poleas, del acoplamiento al husillo y de

Commit message: [E1] El motor de d3 pasa a vertical
Una correa dentada exige ejes paralelos, y el motor tumbado quedaba a noventa
grados del husillo. Se coloca vertical sobre el eslabon 2, a 30 mm del codo,
lo que deja 110 mm entre centros de polea.

Ocupa z de 162 a 254 mm, por debajo de la cima del husillo, de modo que la
altura de la estacion sigue siendo 307 mm. El tensor de inercia del eslabon 2
se recalcula con el cilindro orientado segun Z.

File: src/station1_description/urdf/parametros.xacro (robot description, xacro)
@@ -116,4 +116,8 @@
   <!-- Posicion del motor de theta2 en la base, junto a la columna -->
   <xacro:property name="motor2_offset" value="0.060"/>
+  <!-- Posicion del motor de d3 sobre el eslabon 2, medida desde el codo.
+       Va vertical, paralelo al husillo, porque una correa dentada exige
+       ejes paralelos. La distancia entre centros es l2 - motor3_offset. -->
+  <xacro:property name="motor3_offset" value="0.030"/>
   <!-- Eslabones del brazo: acrilico cortado por laser, 8 mm -->
   <xacro:property name="brazo_ancho"   value="0.050"/>

File: src/station1_description/urdf/station1.urdf.xacro (robot description, xacro)
@@ -122,6 +122,9 @@
   </joint>
   <!-- link_2: pletina, motor de d3 sobre el codo y husillo en el extremo.
-       Es el unico eslabon que carga un motor, y va en el codo y no en el
-       extremo para reducir su brazo respecto del eje de theta1. -->
+       Es el unico eslabon que carga un motor, y va junto al codo y no en el
+       extremo para reducir su brazo respecto del eje de theta1.
+       El motor va vertical, paralelo al husillo: una correa dentada exige
+       ejes paralelos. La distancia entre centros de las poleas es la que
+       separa el motor del husillo. -->
   <xacro:property name="m_barra2"   value="${densidad_acrilico * l2 * brazo_ancho * brazo_espesor}"/>
   <xacro:property name="m_husillo"  value="${densidad_acero * pi * husillo_radio * husillo_radio * husillo_largo}"/>
@@ -129,6 +132,6 @@
   <!-- Posiciones de cada cuerpo dentro del eslabon -->
   <xacro:property name="cx_barra2"  value="${l2/2}"/>
-  <xacro:property name="cx_motor2"  value="${motor_largo/2 + 0.010}"/>
-  <xacro:property name="cz_motor2"  value="${brazo_espesor/2 + motor_diametro/2}"/>
+  <xacro:property name="cx_motor2"  value="${motor3_offset}"/>
+  <xacro:property name="cz_motor2"  value="${brazo_espesor/2 + motor_largo/2}"/>
   <xacro:property name="cx_husillo" value="${l2}"/>
   <xacro:property name="cz_husillo" value="${husillo_largo/2}"/>
@@ -152,5 +155,5 @@
     </visual>
     <visual>
-      <origin xyz="${cx_motor2} 0 ${cz_motor2}" rpy="0 ${pi/2} 0"/>
+      <origin xyz="${cx_motor2} 0 ${cz_motor2}"/>
       <geometry><cylinder radius="${motor_diametro/2}" length="${motor_largo}"/></geometry>
       <material name="motor"/>
@@ -166,5 +169,5 @@
     </collision>
     <collision>
-      <origin xyz="${cx_motor2} 0 ${cz_motor2}" rpy="0 ${pi/2} 0"/>
+      <origin xyz="${cx_motor2} 0 ${cz_motor2}"/>
       <geometry><cylinder radius="${motor_diametro/2}" length="${motor_largo}"/></geometry>
     </collision>
@@ -174,5 +177,5 @@
       <inertia
         ixx="${ m_barra2*(brazo_ancho*brazo_ancho + brazo_espesor*brazo_espesor)/12.0 + m_barra2*dz_b*dz_b
-              + motor_masa*(motor_diametro/2)*(motor_diametro/2)/2.0 + motor_masa*dz_m*dz_m
+              + motor_masa*(3*(motor_diametro/2)*(motor_diametro/2) + motor_largo*motor_largo)/12.0 + motor_masa*dz_m*dz_m
               + m_husillo*(3*husillo_radio*husillo_radio + husillo_largo*husillo_largo)/12.0 + m_husillo*dz_h*dz_h }"
         ixy="0.0"
@@ -183,5 +186,5 @@
         iyz="0.0"
         izz="${ m_barra2*(l2*l2 + brazo_ancho*brazo_ancho)/12.0 + m_barra2*dx_b*dx_b
-              + motor_masa*(3*(motor_diametro/2)*(motor_diametro/2) + motor_largo*motor_largo)/12.0 + motor_masa*dx_m*dx_m
+              + motor_masa*(motor_diametro/2)*(motor_diametro/2)/2.0 + motor_masa*dx_m*dx_m
               + m_husillo*(husillo_radio*husillo_radio)/2.0 + m_husillo*dx_h*dx_h }"/>
     </inertial>

Commit message: [E1] El motor de theta2 pasa al eslabon 1, coaxial con theta1
Con el motor en la base y descentrado, la distancia entre su polea y la del
codo cambiaria al girar theta1, porque el codo va montado en el eslabon 1: la
correa no puede trabajar asi.

Montado sobre el eslabon 1 y coaxial con el eje de theta1, la distancia entre
centros es constante e igual a l1, y no aparece acoplamiento cinematico entre
las dos articulaciones. Su masa gira con el brazo pero a radio cero, de modo
que solo aporta su propio momento polar.

El eslabon 1 pasa de 125 a 335 g con inercia compuesta.

File: src/station1_description/urdf/parametros.xacro (robot description, xacro)
@@ -114,6 +114,7 @@
   <!-- Columna: tubo que aloja el motor de theta1 -->
   <xacro:property name="columna_radio" value="0.030"/>
-  <!-- Posicion del motor de theta2 en la base, junto a la columna -->
-  <xacro:property name="motor2_offset" value="0.060"/>
+  <!-- El motor de theta2 va sobre el eslabon 1, coaxial con el eje de
+       theta1, de modo que la distancia a la polea del codo sea constante
+       al girar el brazo. Su masa queda a radio cero del eje de theta1. -->
   <!-- Posicion del motor de d3 sobre el eslabon 2, medida desde el codo.
        Va vertical, paralelo al husillo, porque una correa dentada exige

File: src/station1_description/urdf/station1.urdf.xacro (robot description, xacro)
@@ -10,5 +10,5 @@
   masa en voladizo:
     theta1  motor alojado dentro de la columna, accionamiento directo
-    theta2  motor en la base, correa dentada por dentro del eslabon 1
+    theta2  motor sobre el eslabon 1 y coaxial con theta1, correa al codo
     d3      motor en el codo, correa al husillo del extremo del eslabon 2
   Dos de los tres motores quedan fijos a la base y no cargan el brazo.
@@ -30,5 +30,5 @@
   <material name="motor">     <color rgba="0.20 0.20 0.22 1.0"/></material>
   <!-- ==================================================================
-       base_link: placa de MDF, columna y los dos motores rotacionales.
+       base_link: placa de MDF, columna y el motor de theta1 en su interior.
        Es un eslabon fijo al mundo, de modo que su inercia no interviene en
        la dinamica; se declara con la masa real para que el balance total de
@@ -37,5 +37,5 @@
   <xacro:property name="m_placa"   value="${densidad_mdf * base_x * base_y * base_z}"/>
   <xacro:property name="m_columna" value="${densidad_pla * pi * columna_radio * columna_radio * (altura_columna - base_z)}"/>
-  <xacro:property name="m_base"    value="${m_placa + m_columna + 2 * motor_masa}"/>
+  <xacro:property name="m_base"    value="${m_placa + m_columna + motor_masa}"/>
   <link name="${p}base_link">
     <visual>
@@ -49,11 +49,4 @@
       <material name="pla"/>
     </visual>
-    <!-- Motor de theta2, en la base junto a la columna. Acciona el codo por
-         correa; su masa nunca viaja con el brazo. -->
-    <visual>
-      <origin xyz="${motor2_offset} 0 ${base_z + motor_largo/2}"/>
-      <geometry><cylinder radius="${motor_diametro/2}" length="${motor_largo}"/></geometry>
-      <material name="motor"/>
-    </visual>
     <collision>
       <origin xyz="0 0 ${base_z/2}"/>
@@ -63,8 +56,4 @@
       <origin xyz="0 0 ${base_z + (altura_columna - base_z)/2}"/>
       <geometry><cylinder radius="${columna_radio}" length="${altura_columna - base_z}"/></geometry>
-    </collision>
-    <collision>
-      <origin xyz="${motor2_offset} 0 ${base_z + motor_largo/2}"/>
-      <geometry><cylinder radius="${motor_diametro/2}" length="${motor_largo}"/></geometry>
     </collision>
     <inertial>
@@ -87,7 +76,14 @@
     <dynamics damping="0.05" friction="0.01"/>
   </joint>
-  <!-- link_1: pletina de acrilico mas las dos poleas de la correa de theta2 -->
+  <!-- link_1: pletina de acrilico, las dos poleas de la correa de theta2 y el
+       propio motor de theta2, montado sobre el eje de giro. Al estar a radio
+       cero, su masa apenas contribuye a la inercia del eslabon. -->
   <xacro:property name="m_barra1" value="${densidad_acrilico * l1 * brazo_ancho * brazo_espesor}"/>
-  <xacro:property name="m_link1"  value="${m_barra1 + 2 * polea_masa}"/>
+  <xacro:property name="m_link1"  value="${m_barra1 + 2 * polea_masa + motor_masa}"/>
+  <xacro:property name="cz_motor1" value="${brazo_espesor/2 + motor_largo/2}"/>
+  <xacro:property name="cx_link1"
+    value="${(m_barra1*(l1/2) + 2*polea_masa*(l1/2)) / m_link1}"/>
+  <xacro:property name="cz_link1"
+    value="${motor_masa*cz_motor1 / m_link1}"/>
   <link name="${p}link_1">
     <visual>
@@ -100,13 +96,30 @@
       <geometry><box size="${l1} ${brazo_ancho} ${brazo_espesor}"/></geometry>
     </collision>
-    <!-- Las poleas van en los dos extremos, de modo que el centro de masa
-         del conjunto sigue estando a media longitud. -->
-    <inertial>
-      <origin xyz="${l1/2} 0 0"/>
+    <visual>
+      <origin xyz="0 0 ${cz_motor1}"/>
+      <geometry><cylinder radius="${motor_diametro/2}" length="${motor_largo}"/></geometry>
+      <material name="motor"/>
+    </visual>
+    <collision>
+      <origin xyz="0 0 ${cz_motor1}"/>
+      <geometry><cylinder radius="${motor_diametro/2}" length="${motor_largo}"/></geometry>
+    </collision>
+    <inertial>
+      <origin xyz="${cx_link1} 0 ${cz_link1}"/>
       <mass value="${m_link1}"/>
       <inertia
-        ixx="${m_barra1*(brazo_ancho*brazo_ancho + brazo_espesor*brazo_espesor)/12.0}" ixy="0.0" ixz="0.0"
-        iyy="${m_barra1*(l1*l1 + brazo_espesor*brazo_espesor)/12.0 + 2*polea_masa*(l1/2)*(l1/2)}" iyz="0.0"
-        izz="${m_barra1*(l1*l1 + brazo_ancho*brazo_ancho)/12.0 + 2*polea_masa*(l1/2)*(l1/2)}"/>
+        ixx="${ m_barra1*(brazo_ancho*brazo_ancho + brazo_espesor*brazo_espesor)/12.0 + m_barra1*cz_link1*cz_link1
+              + motor_masa*(3*(motor_diametro/2)*(motor_diametro/2) + motor_largo*motor_largo)/12.0
+              + motor_masa*(cz_motor1-cz_link1)*(cz_motor1-cz_link1) }"
+        ixy="0.0"
+        ixz="${ -( m_barra1*(l1/2-cx_link1)*(-cz_link1) + motor_masa*(0-cx_link1)*(cz_motor1-cz_link1) ) }"
+        iyy="${ m_barra1*(l1*l1 + brazo_espesor*brazo_espesor)/12.0 + m_barra1*((l1/2-cx_link1)*(l1/2-cx_link1) + cz_link1*cz_link1)
+              + 2*polea_masa*(l1/2)*(l1/2)
+              + motor_masa*(3*(motor_diametro/2)*(motor_diametro/2) + motor_largo*motor_largo)/12.0
+              + motor_masa*(cx_link1*cx_link1 + (cz_motor1-cz_link1)*(cz_motor1-cz_link1)) }"
+        iyz="0.0"
+        izz="${ m_barra1*(l1*l1 + brazo_ancho*brazo_ancho)/12.0 + m_barra1*(l1/2-cx_link1)*(l1/2-cx_link1)
+              + 2*polea_masa*(l1/2)*(l1/2)
+              + motor_masa*(motor_diametro/2)*(motor_diametro/2)/2.0 + motor_masa*cx_link1*cx_link1 }"/>
     </inertial>
   </link>

Commit message: entrega 2

File: src/station1_description/urdf/parametros.xacro (robot description, xacro)
@@ -31,6 +31,11 @@
   <!-- ================== Restricciones de la guia ================== -->
   <!-- Envolvente de trabajo en el plano XY: radio 320 mm +/- 20 mm.   -->
-  <!-- Envolvente en el plano YZ: 300 mm +/- 20 mm, interpretado como  -->
-  <!-- la altura total de la estacion. Confirmar con el profesor.      -->
+  <!-- Envolvente en el plano YZ: la guia lo enuncia como 300 mm +/- 20, -->
+  <!-- es decir de 280 a 320, y se lee como la altura total. El profesor  -->
+  <!-- aclaro el 16/08/2026 que admitia leerse como 320 +/- 20, pero se   -->
+  <!-- dimensiono con el criterio escrito, que es el mas estricto de los  -->
+  <!-- dos, de modo que cumple bajo cualquiera de las dos lecturas.       -->
+  <!-- La estacion mide 307, con el extremo del husillo como punto mas    -->
+  <!-- alto: quedan 13 mm de margen bajo el techo de 320.                 -->
   <xacro:property name="alcance_xy"      value="0.320"/>
   <xacro:property name="altura_estacion" value="0.307"/>

File: src/station1_description/urdf/station1.urdf.xacro (robot description, xacro)
@@ -23,4 +23,10 @@
   <xacro:include filename="$(find station1_description)/urdf/inercias.xacro"/>
   <xacro:include filename="$(find station1_description)/urdf/station1.gazebo.xacro"/>
+  <xacro:include filename="$(find station1_description)/urdf/station1.ros2_control.xacro"/>
+  <!-- Con control:=false el modelo se puede abrir en RViz sin levantar el
+       controller_manager, que es como se reviso el arbol TF en la Entrega 1. -->
+  <xacro:arg name="control" default="true"/>
+  <xacro:arg name="controladores"
+             default="$(find station1_description)/config/station1_controllers.yaml"/>
   <material name="acrilico">  <color rgba="0.35 0.55 0.75 0.75"/></material>
   <material name="mdf">       <color rgba="0.72 0.58 0.38 1.0"/></material>
@@ -261,5 +267,19 @@
     <limit lower="0.0" upper="${carrera_d3}"
            velocity="${vel_pris}" effort="${esfuerzo_pris}"/>
-    <dynamics damping="2.0" friction="0.5"/>
+    <!-- La friccion no es un numero de relleno: es lo que hace del eje un eje
+         autoblocante. El husillo trabaja con un rendimiento directo de 0.2, y
+         un husillo por debajo de 0.5 no se puede retroaccionar: el carro no
+         baja solo aunque se corte la corriente. Con 0.5 N, por debajo de los
+         2.17 N que pesa el conjunto, se describia justo lo contrario, un eje
+         que se descuelga. Con 4.0 N, por encima del peso, el eje se sostiene
+         solo y al actuador le quedan 61 N para moverlo.
+         Aviso para no atribuirle lo que no hace: este cambio NO es lo que
+         arreglo el error de seguimiento de la prismatica al descender. Ese
+         error resulto depender de la velocidad pedida, no de la gravedad, y se
+         corrigio planificando al 70 % del limite de velocidad; la medida esta
+         en station1_control/trayectoria.py. La gravedad si explica que
+         bajando el error sea unas diez veces mayor que subiendo a igualdad de
+         velocidad, pero no el fenomeno principal. -->
+    <dynamics damping="2.0" friction="4.0"/>
   </joint>
   <!-- ==================================================================
@@ -341,11 +361,41 @@
     </xacro:inercia_componente>
   </link>
-  <!-- Punto de referencia del efector, donde se sujeta la pieza. -->
+  <!-- Punto de referencia del efector, donde se sujeta la pieza.
+       Cuelga del carro y no de la mordaza: tool0 es un sistema fijo del
+       brazo, y si girase con el servo el punto de trabajo se desplazaria
+       16.8 mm al abrir la pinza y el grupo de planificacion pasaria a tener
+       cuatro articulaciones en lugar de los tres grados de libertad que pide
+       la guia. Con la mordaza cerrada la pose es identica a la de la
+       Entrega 1. -->
   <joint name="${p}tool0_joint" type="fixed">
-    <parent link="${p}gripper_link"/>
+    <parent link="${p}link_3"/>
     <child  link="${p}tool0"/>
-    <origin xyz="0 0 ${-gripper_z}"/>
+    <origin xyz="0 0 ${-(vastago_largo + gripper_z)}"/>
   </joint>
   <link name="${p}tool0"/>
   <xacro:station1_gazebo prefijo="${p}"/>
+  <!-- ==================================================================
+       Acople cinematico de la pieza, segun ADR-002.
+       No acopla al arrancar. El nodo de la estacion pide el acople cuando
+       cierra la mordaza sobre la pieza y lo deshace antes de abrirla.
+  =================================================================== -->
+  <xacro:arg name="acople" default="true"/>
+  <xacro:arg name="pieza" default="pieza"/>
+  <xacro:if value="$(arg acople)">
+    <gazebo>
+      <plugin filename="gz-sim-detachable-joint-system"
+              name="gz::sim::systems::DetachableJoint">
+        <parent_link>${p}gripper_link</parent_link>
+        <child_model>$(arg pieza)</child_model>
+        <child_link>cuerpo</child_link>
+        <attach_topic>/station1/pieza/attach</attach_topic>
+        <detach_topic>/station1/pieza/detach</detach_topic>
+        <suppress_child_warning>true</suppress_child_warning>
+      </plugin>
+    </gazebo>
+  </xacro:if>
+  <xacro:if value="$(arg control)">
+    <xacro:station1_ros2_control prefijo="${p}"
+                                 controladores="$(arg controladores)"/>
+  </xacro:if>
 </robot>
