Commit message: station3_description: colores del robot en el URDF (base blanca, Link1_1 y Link2_1 amarillo de maquinaria, Prismatico_1 negro). El material silver queda definido sin uso. Verificado en Gazebo a ojo; no se comprobo si las etiquetas Gazebo/Silver de station3.gazebo.xacro pisan estos colores

File: src/station3_description/urdf/station3.urdf.xacro (robot description, xacro)
@@ -19,4 +19,13 @@
     <color rgba="0.700 0.700 0.700 1.000"/>
   </material>
+  <material name="blanco">
+    <color rgba="0.950 0.950 0.950 1.000"/>
+  </material>
+  <material name="amarillo_maquinaria">
+    <color rgba="1.000 0.780 0.050 1.000"/>
+  </material>
+  <material name="negro">
+    <color rgba="0.050 0.050 0.050 1.000"/>
+  </material>
   <link name="${p}base_link">
     <inertial>
@@ -28,5 +37,5 @@
         <mesh filename="package://station3_description/meshes/base_link.stl" scale="0.001 0.001 0.001"/>
       </geometry>
-      <material name="silver"/>
+      <material name="blanco"/>
     </visual>
     <collision>
@@ -46,5 +55,5 @@
         <mesh filename="package://station3_description/meshes/Link1_1.stl" scale="0.001 0.001 0.001"/>
       </geometry>
-      <material name="silver"/>
+      <material name="amarillo_maquinaria"/>
     </visual>
     <collision>
@@ -64,5 +73,5 @@
         <mesh filename="package://station3_description/meshes/Link2_1.stl" scale="0.001 0.001 0.001"/>
       </geometry>
-      <material name="silver"/>
+      <material name="amarillo_maquinaria"/>
     </visual>
     <collision>
@@ -82,5 +91,5 @@
         <mesh filename="package://station3_description/meshes/Prismatico_1.stl" scale="0.001 0.001 0.001"/>
       </geometry>
-      <material name="silver"/>
+      <material name="negro"/>
     </visual>
     <collision>
