Commit message: station2_description: visual con las mallas STL del CAD v5.7 (normales recalculadas), primitivas de la base orientadas como el CAD (PCB en +x, motor de theta1 en -y), display centrado en el origen y en reposo; capturas y prueba_estacion (3/3) regeneradas
Co-Authored-By: Claude Opus 5.5 (1M context) <noreply@anthropic.com>

File: src/station2_description/urdf/station2.urdf.xacro (robot description, xacro)
@@ -15,6 +15,8 @@
   Camara: Raspberry Pi Camera Module 3 Wide bajo el eslabon 2.
   Todos los frames llevan el prefijo de la estacion, segun ADR-005.
-  Geometria de colision simplificada a cajas y cilindros. Las mallas del CAD,
-  cuando esten en meshes/, solo sustituyen la parte visual.
+  Visual con las mallas STL del CAD v5.7 (meshes/, exportadas de Fusion por
+  cad/station2/urdf_cad/scripts/mallas_fusion.py en la pose cero, en metros y
+  en el marco de cada eslabon). Con mallas:=false se vuelve a los solidos
+  simples. La colision sigue siendo de cajas y cilindros.
 -->
 <robot xmlns:xacro="http://www.ros.org/wiki/xacro" name="station2">
@@ -33,4 +35,6 @@
        de render; con camara:=false el modelo queda igual pero sin sensor. -->
   <xacro:arg name="camara" default="true"/>
+  <!-- Visual con las mallas del CAD (true) o con solidos simples (false). -->
+  <xacro:arg name="mallas" default="true"/>
   <material name="acrilico"> <color rgba="0.85 0.88 0.92 0.80"/></material>
   <material name="acrilico_negro"> <color rgba="0.10 0.10 0.12 1.0"/></material>
@@ -39,4 +43,21 @@
   <material name="motor">    <color rgba="0.20 0.20 0.22 1.0"/></material>
   <material name="pcb">      <color rgba="0.05 0.35 0.15 1.0"/></material>
+  <material name="cad_base"> <color rgba="0.78 0.82 0.88 1.0"/></material>
+  <material name="cad_brazo"><color rgba="0.93 0.76 0.20 1.0"/></material>
+  <material name="cad_mordaza"><color rgba="0.92 0.92 0.92 1.0"/></material>
+  <!-- Visual con la malla del CAD; el origen va en el marco del eslabon.
+       Ruta file:// absoluta (la resuelve xacro): asi la encuentran RViz y
+       Gazebo sin tocar GZ_SIM_RESOURCE_PATH, tambien cuando la estacion se
+       anade al Gazebo de la Estacion 1 (simulacion_en_linea.launch.py). -->
+  <xacro:property name="ruta_mallas" value="file://$(find station2_description)/meshes"/>
+  <xacro:macro name="malla" params="nombre material xyz:='0 0 0'">
+    <visual>
+      <origin xyz="${xyz}"/>
+      <geometry>
+        <mesh filename="${ruta_mallas}/${nombre}.stl"/>
+      </geometry>
+      <material name="${material}"/>
+    </visual>
+  </xacro:macro>
   <!-- Alturas derivadas -->
   <xacro:property name="z_base_sup" value="${patas_z + base_z}"/>
@@ -47,8 +68,13 @@
        base_link: placa de acrilico de 300 x 300 sobre patas de goma, torre
        en cajon de acrilico con el lazy susan de theta1 arriba, motor de
-       theta1 en el piso por detras y la PCB de control en la zona +y.
+       theta1 en el piso por detras (-y) y la PCB de control en la zona +x,
+       como en el CAD.
        Es fijo al mundo; su masa cuenta para el balance de la estacion.
   =================================================================== -->
   <link name="${p}base_link">
+    <xacro:if value="$(arg mallas)">
+      <xacro:malla nombre="base_link" material="cad_base"/>
+    </xacro:if>
+    <xacro:unless value="$(arg mallas)">
     <visual>
       <origin xyz="0 0 ${patas_z + base_z/2}"/>
@@ -61,16 +87,17 @@
       <material name="acrilico"/>
     </visual>
-    <!-- Motor de theta1 en el piso, 59 mm por detras del eje -->
-    <visual>
-      <origin xyz="-0.059 0 ${z_base_sup + motor_largo/2}"/>
+    <!-- Motor de theta1 en el piso, 59 mm por detras del eje (-y) -->
+    <visual>
+      <origin xyz="0 -0.059 ${z_base_sup + motor_largo/2}"/>
       <geometry><cylinder radius="${motor_diametro/2}" length="${motor_largo}"/></geometry>
       <material name="motor"/>
     </visual>
-    <!-- PCB de control, 100 x 99 mm, sobre separadores en la zona +y -->
-    <visual>
-      <origin xyz="0 0.095 ${z_base_sup + 0.012}"/>
-      <geometry><box size="0.100 0.099 0.002"/></geometry>
+    <!-- PCB de control, 99.8 x 98.7 mm, sobre separadores en la zona +x -->
+    <visual>
+      <origin xyz="0.095 0 ${z_base_sup + 0.012}"/>
+      <geometry><box size="0.099 0.100 0.002"/></geometry>
       <material name="pcb"/>
     </visual>
+    </xacro:unless>
     <collision>
       <origin xyz="0 0 ${(patas_z + base_z)/2}"/>
@@ -121,4 +148,8 @@
   =================================================================== -->
   <link name="${p}link_1">
+    <xacro:if value="$(arg mallas)">
+      <xacro:malla nombre="link_1" material="cad_brazo"/>
+    </xacro:if>
+    <xacro:unless value="$(arg mallas)">
     <visual>
       <origin xyz="${(l1+2*cola)/2 - cola} 0 ${brazo_espesor/2}"/>
@@ -131,4 +162,5 @@
       <material name="motor"/>
     </visual>
+    </xacro:unless>
     <collision>
       <origin xyz="${(l1+2*cola)/2 - cola} 0 ${brazo_espesor/2}"/>
@@ -159,4 +191,8 @@
   =================================================================== -->
   <link name="${p}link_2">
+    <xacro:if value="$(arg mallas)">
+      <xacro:malla nombre="link_2" material="cad_brazo"/>
+    </xacro:if>
+    <xacro:unless value="$(arg mallas)">
     <visual>
       <origin xyz="${(l2+2*cola)/2 - cola} 0 ${brazo_espesor/2}"/>
@@ -191,4 +227,5 @@
       <material name="pcb"/>
     </visual>
+    </xacro:unless>
     <collision>
       <origin xyz="${(l2+2*cola)/2 - cola} 0 ${brazo_espesor/2}"/>
@@ -224,4 +261,8 @@
   =================================================================== -->
   <link name="${p}link_3">
+    <xacro:if value="$(arg mallas)">
+      <xacro:malla nombre="link_3" material="cad_mordaza"/>
+    </xacro:if>
+    <xacro:unless value="$(arg mallas)">
     <visual>
       <origin xyz="0 0 ${dedo_largo + pinza_z + largo_vastago/2}"/>
@@ -234,4 +275,5 @@
       <material name="pla"/>
     </visual>
+    </xacro:unless>
     <collision>
       <origin xyz="0 0 ${dedo_largo + pinza_z/2}"/>
@@ -258,4 +300,11 @@
     </joint>
     <link name="${p}${nombre}">
+      <!-- La malla esta en el marco de link_3 (pinza abierta): se deshace
+           el desplazamiento del origen del dedo. -->
+      <xacro:if value="$(arg mallas)">
+        <xacro:malla nombre="${nombre}" material="cad_mordaza"
+                     xyz="0 ${-signo * (luz_abierta/2 + dedo_y/2)} 0"/>
+      </xacro:if>
+      <xacro:unless value="$(arg mallas)">
       <visual>
         <origin xyz="0 0 ${dedo_largo/2 - dedo_bajo_tool}"/>
@@ -263,4 +312,5 @@
         <material name="pla"/>
       </visual>
+      </xacro:unless>
       <collision>
         <origin xyz="0 0 ${dedo_largo/2 - dedo_bajo_tool}"/>

Commit message: station2_description: mallas del CAD v5.7 con colores y materiales sacadas del STEP (Collada; acrilico transparente en eslabones solo visuales *_acrilico), grabado laser de la base visible; scripts de conversion; capturas y prueba_estacion (3/3) regeneradas
Co-Authored-By: Claude Opus 5.5 (1M context) <noreply@anthropic.com>

File: src/station2_description/urdf/station2.urdf.xacro (robot description, xacro)
@@ -15,8 +15,11 @@
   Camara: Raspberry Pi Camera Module 3 Wide bajo el eslabon 2.
   Todos los frames llevan el prefijo de la estacion, segun ADR-005.
-  Visual con las mallas STL del CAD v5.7 (meshes/, exportadas de Fusion por
-  cad/station2/urdf_cad/scripts/mallas_fusion.py en la pose cero, en metros y
-  en el marco de cada eslabon). Con mallas:=false se vuelve a los solidos
-  simples. La colision sigue siendo de cajas y cilindros.
+  Visual con las mallas del CAD v5.7 con los colores de cada pieza (meshes/,
+  sacadas del STEP del ensamble por scripts/step_a_mallas.py y
+  scripts/mallas_dae.py, en la pose cero, en metros y en el marco de cada
+  eslabon): Collada para las piezas opacas y STL para el acrilico, que va en
+  un eslabon solo visual *_acrilico con color transparente. Con
+  mallas:=false se vuelve a los solidos simples. La colision sigue siendo de
+  cajas y cilindros.
 -->
 <robot xmlns:xacro="http://www.ros.org/wiki/xacro" name="station2">
@@ -43,20 +46,40 @@
   <material name="motor">    <color rgba="0.20 0.20 0.22 1.0"/></material>
   <material name="pcb">      <color rgba="0.05 0.35 0.15 1.0"/></material>
-  <material name="cad_base"> <color rgba="0.78 0.82 0.88 1.0"/></material>
-  <material name="cad_brazo"><color rgba="0.93 0.76 0.20 1.0"/></material>
-  <material name="cad_mordaza"><color rgba="0.92 0.92 0.92 1.0"/></material>
-  <!-- Visual con la malla del CAD; el origen va en el marco del eslabon.
+  <!-- Acrilico claro de corte laser, como el 'Acrilico, claro' de Fusion. -->
+  <material name="acrilico_claro"><color rgba="0.82 0.91 0.96 0.35"/></material>
+  <!-- Visual con la malla del CAD (Collada con los colores y materiales de
+       cada pieza); el origen va en el marco del eslabon.
        Ruta file:// absoluta (la resuelve xacro): asi la encuentran RViz y
        Gazebo sin tocar GZ_SIM_RESOURCE_PATH, tambien cuando la estacion se
        anade al Gazebo de la Estacion 1 (simulacion_en_linea.launch.py). -->
   <xacro:property name="ruta_mallas" value="file://$(find station2_description)/meshes"/>
-  <xacro:macro name="malla" params="nombre material xyz:='0 0 0'">
+  <xacro:macro name="malla" params="nombre xyz:='0 0 0'">
     <visual>
       <origin xyz="${xyz}"/>
       <geometry>
-        <mesh filename="${ruta_mallas}/${nombre}.stl"/>
+        <mesh filename="${ruta_mallas}/${nombre}.dae"/>
       </geometry>
-      <material name="${material}"/>
-    </visual>
+      <!-- Sin <material>: los colores van en la malla (uno por pieza). -->
+    </visual>
+  </xacro:macro>
+  <!-- Piezas de acrilico de cada eslabon, en un eslabon solo visual unido con
+       una junta fija. RViz no lee la opacidad de las mallas Collada y aplica
+       una sola opacidad a todo el eslabon, asi que el acrilico transparente
+       necesita su propio eslabon. Sin inercia: Gazebo lo funde con el padre. -->
+  <xacro:macro name="acrilico" params="nombre xyz:='0 0 0'">
+    <joint name="${p}${nombre}_acrilico_joint" type="fixed">
+      <parent link="${p}${nombre}"/>
+      <child  link="${p}${nombre}_acrilico"/>
+      <origin xyz="0 0 0"/>
+    </joint>
+    <link name="${p}${nombre}_acrilico">
+      <visual>
+        <origin xyz="${xyz}"/>
+        <geometry>
+          <mesh filename="${ruta_mallas}/${nombre}_acrilico.stl"/>
+        </geometry>
+        <material name="acrilico_claro"/>
+      </visual>
+    </link>
   </xacro:macro>
   <!-- Alturas derivadas -->
@@ -74,5 +97,5 @@
   <link name="${p}base_link">
     <xacro:if value="$(arg mallas)">
-      <xacro:malla nombre="base_link" material="cad_base"/>
+      <xacro:malla nombre="base_link"/>
     </xacro:if>
     <xacro:unless value="$(arg mallas)">
@@ -110,4 +133,7 @@
     <xacro:inercia_cad masa="${m_base}" centro="${c_base}" tensor="${i_base}"/>
   </link>
+  <xacro:if value="$(arg mallas)">
+    <xacro:acrilico nombre="base_link"/>
+  </xacro:if>
   <!-- ==================================================================
        Anclaje al mundo. En la maquina real no hay tornillos a la mesa: el
@@ -149,5 +175,5 @@
   <link name="${p}link_1">
     <xacro:if value="$(arg mallas)">
-      <xacro:malla nombre="link_1" material="cad_brazo"/>
+      <xacro:malla nombre="link_1"/>
     </xacro:if>
     <xacro:unless value="$(arg mallas)">
@@ -173,4 +199,7 @@
     <xacro:inercia_cad masa="${m_link1}" centro="${c_link1}" tensor="${i_link1}"/>
   </link>
+  <xacro:if value="$(arg mallas)">
+    <xacro:acrilico nombre="link_1"/>
+  </xacro:if>
   <!-- ==================== theta2: codo ====================
        El origen esta en la cara inferior del eslabon 2, por encima del
@@ -192,5 +221,5 @@
   <link name="${p}link_2">
     <xacro:if value="$(arg mallas)">
-      <xacro:malla nombre="link_2" material="cad_brazo"/>
+      <xacro:malla nombre="link_2"/>
     </xacro:if>
     <xacro:unless value="$(arg mallas)">
@@ -242,4 +271,7 @@
     <xacro:inercia_cad masa="${m_link2}" centro="${c_link2}" tensor="${i_link2}"/>
   </link>
+  <xacro:if value="$(arg mallas)">
+    <xacro:acrilico nombre="link_2"/>
+  </xacro:if>
   <!-- ==================== d3: desplazamiento vertical ====================
        El origen de link_3 es tool0 con d3 = 0, el punto de trabajo en lo
@@ -262,5 +294,5 @@
   <link name="${p}link_3">
     <xacro:if value="$(arg mallas)">
-      <xacro:malla nombre="link_3" material="cad_mordaza"/>
+      <xacro:malla nombre="link_3"/>
     </xacro:if>
     <xacro:unless value="$(arg mallas)">
@@ -286,4 +318,7 @@
     <xacro:inercia_cad masa="${m_link3}" centro="${c_link3}" tensor="${i_link3}"/>
   </link>
+  <xacro:if value="$(arg mallas)">
+    <xacro:acrilico nombre="link_3"/>
+  </xacro:if>
   <!-- ==================== Mordaza: dos dedos prismaticos ====================
        No son grados de libertad del brazo: los mueve el servo por el piñon y
@@ -303,5 +338,5 @@
            el desplazamiento del origen del dedo. -->
       <xacro:if value="$(arg mallas)">
-        <xacro:malla nombre="${nombre}" material="cad_mordaza"
+        <xacro:malla nombre="${nombre}"
                      xyz="0 ${-signo * (luz_abierta/2 + dedo_y/2)} 0"/>
       </xacro:if>
@@ -321,4 +356,7 @@
       </xacro:inercia_componente>
     </link>
+    <xacro:if value="$(arg mallas)">
+      <xacro:acrilico nombre="${nombre}" xyz="0 ${-signo * (luz_abierta/2 + dedo_y/2)} 0"/>
+    </xacro:if>
   </xacro:macro>
   <xacro:dedo nombre="dedo_1" signo="1"/>
